File: kicad/SCCS-RPI.kicad_sch (KiCad schematic)
At the start: 59 parts, among them J1 Conn_Coaxial, J2 12VDC IN, U1 AP64501SP-13

Commit message: Updated Kicad schematics
Parts:
- removed C24: 100uF, Capacitor_SMD:C_0805_2012Metric, symbol Device:C_Small
- added C24: 100uF, Capacitor_THT:CP_Radial_D6.3mm_P2.50mm, symbol Device:C_Polarized_Small
- C23: LCSC Part # C17342103 -> C541516
- C3: value 47uF -> 22uF; LCSC Part # C380345 -> C86816
- J1: footprint Connector_Coaxial:U.FL_Hirose_U.FL-R-SMT-1_Vertical -> Connector_Coaxial:SMA_Amphenol_132134-11_Vertical; LCSC Part # C88373 -> C20415804
Connections:
- net +3V3: now also R5.1
- net GND: now also C24.2; no longer R5.1
- net at R12.2: now also C24.1
