File: kicad/analog_inputs.kicad_sch (KiCad schematic)
At the start: 5 parts

Commit message: Updated Kicad schematics
Parts:
- removed R18: 470R, Resistor_SMD:R_0805_2012Metric, symbol Device:R
Connections:
- net at FB2.1: now also i4.1 (Pin_1)
Changed lines of the file:
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@@
-	(wire
-		(pts
-			(xy 95.25 69.85) (xy 100.33 69.85)
-		)
-		(stroke
-			(width 0)
-			(type default)
-		)
-	)
 	(wire
 		(pts
@@
 		(pts
 			(xy 119.38 71.12) (xy 119.38 69.85)
+		)
+		(stroke
+			(width 0)
+			(type default)
+		)
+	)
+	(wire
+		(pts
+			(xy 87.63 69.85) (xy 100.33 69.85)
 		)
 		(stroke
@@
 				(path "/ce21946f-7655-4864-b48a-50deff8538eb/f275b187-1ecf-4da8-9601-a32837f11b2b"
 					(reference "FB4")
-					(unit 1)
-				)
-			)
-		)
-	)
-	(symbol
-		(lib_id "Device:R")
-		(at 91.44 69.85 90)
-		(unit 1)
-		(body_style 1)
-		(exclude_from_sim no)
-		(in_bom yes)
-		(on_board yes)
-		(in_pos_files yes)
-		(dnp no)
-		(property "Reference" "R18"
-			(at 91.44 67.564 90)
-			(show_name no)
-			(do_not_autoplace no)
-			(effects
-				(font
-					(size 1.27 1.27)
-				)
-			)
-		)
-		(property "Value" "470R"
-			(at 91.44 69.85 90)
-			(show_name no)
-			(do_not_autoplace no)
-			(effects
-				(font
-					(size 0.762 0.762)
-				)
-			)
-		)
-		(property "Footprint" "Resistor_SMD:R_0805_2012Metric"
-			(at 91.44 71.628 90)
-			(hide yes)
-			(show_name no)
-			(do_not_autoplace no)
-			(effects
-				(font
-					(size 1.27 1.27)
-				)
-			)
-		)
-		(property "Datasheet" ""
-			(at 91.44 69.85 0)
-			(hide yes)
-			(show_name no)
-			(do_not_autoplace no)
-			(effects
-				(font
-					(size 1.27 1.27)
-				)
-			)
-		)
-		(property "Description" "Resistor"
-			(at 91.44 69.85 0)
-			(hide yes)
-			(show_name no)
-			(do_not_autoplace no)
-			(effects
-				(font
-					(size 1.27 1.27)
-				)
-			)
-		)
-		(property "LCSC Part #" "C17710"
-			(at 91.44 69.85 90)
-			(hide yes)
-			(show_name no)
-			(do_not_autoplace no)
-			(effects
-				(font
-					(size 1.27 1.27)
-				)
-			)
-		)
-		(pin "2"
-		)
-		(pin "1"
-		)
-		(instances
-			(project "SCCS-RPI"
-				(path "/ce21946f-7655-4864-b48a-50deff8538eb/11e9aa4c-c1a1-4a8f-a0a0-7141df7ab674"
-					(reference "R20")
-					(unit 1)
-				)
-				(path "/ce21946f-7655-4864-b48a-50deff8538eb/3114b48f-2d53-4033-bb6c-4b7d97201800"
-					(reference "R18")
-					(unit 1)
-				)
-				(path "/ce21946f-7655-4864-b48a-50deff8538eb/f275b187-1ecf-4da8-9601-a32837f11b2b"
-					(reference "R22")
 					(unit 1)
 				)
@@
 			(project "SCCS-RPI"
 				(path "/ce21946f-7655-4864-b48a-50deff8538eb/11e9aa4c-c1a1-4a8f-a0a0-7141df7ab674"
-					(reference "R19")
+					(reference "R18")
 					(unit 1)
 				)
@@
 				)
 				(path "/ce21946f-7655-4864-b48a-50deff8538eb/f275b187-1ecf-4da8-9601-a32837f11b2b"
-					(reference "R21")
+					(reference "R19")
 					(unit 1)
 				)
@@
 		(dnp no)
 		(fields_autoplaced yes)
-		(property "Reference" "#PWR027"
+		(property "Reference" "#PWR028"
 			(at 99.06 85.09 0)
 			(hide yes)
@@
 			(project "SCCS-RPI"
 				(path "/ce21946f-7655-4864-b48a-50deff8538eb/11e9aa4c-c1a1-4a8f-a0a0-7141df7ab674"
-					(reference "#PWR029")
+					(reference "#PWR030")
 					(unit 1)
 				)
 				(path "/ce21946f-7655-4864-b48a-50deff8538eb/3114b48f-2d53-4033-bb6c-4b7d97201800"
-					(reference "#PWR027")
+					(reference "#PWR028")
 					(unit 1)
 				)
 				(path "/ce21946f-7655-4864-b48a-50deff8538eb/f275b187-1ecf-4da8-9601-a32837f11b2b"
-					(reference "#PWR031")
+					(reference "#PWR032")
 					(unit 1)
 				)
@@
 		(in_pos_files yes)
 		(dnp no)
-		(property "Reference" "#PWR026"
+		(property "Reference" "#PWR027"
 			(at 99.06 66.04 0)
 			(hide yes)
@@
 			(project "SCCS-RPI"
 				(path "/ce21946f-7655-4864-b48a-50deff8538eb/11e9aa4c-c1a1-4a8f-a0a0-7141df7ab674"
-					(reference "#PWR028")
+					(reference "#PWR029")
 					(unit 1)
 				)
 				(path "/ce21946f-7655-4864-b48a-50deff8538eb/3114b48f-2d53-4033-bb6c-4b7d97201800"
-					(reference "#PWR026")
+					(reference "#PWR027")
 					(unit 1)
 				)
 				(path "/ce21946f-7655-4864-b48a-50deff8538eb/f275b187-1ecf-4da8-9601-a32837f11b2b"
-					(reference "#PWR030")
-					(unit 1)
-				)
+					(reference "#PWR031")
+					(unit 1)
+				)
