File: kicad/esp32.kicad_sch (KiCad schematic)
At the start: 8 parts, among them SW1 RESET, SW2 BOOT

Commit message: Updated Kicad schematics
Parts:
- added R36: 10K, Resistor_SMD:R_0402_1005Metric, symbol Device:R
- renumbered C52 to C46, C53 to C47, C54 to C48, C55 to C49, R77 to R37
Connections:
- net +3V3: now also R36.2
- net at ESP32-1.3 (EN), SW1.2: now also R36.1
Other:
- moved on the sheet: SW1
