File: kicad/led_channel.kicad_sch (KiCad schematic)
At the start: 5 parts, among them Q1 IRLB8721PBF

Commit message: Updated Kicad schematics
Parts:
- renumbered D16 to D19, R39 to R40, R40 to R41, R41 to R42
