File: kicad/led_power.kicad_sch (KiCad schematic)
At the start: 3 parts

Commit message: Updated Kicad schematics
Parts:
- renumbered C46 to C54, C47 to C55
Changed lines of the file:
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@@
 		(in_pos_files yes)
 		(dnp no)
-		(property "Reference" "C46"
+		(property "Reference" "C54"
 			(at 96.266 65.024 0)
 			(show_name no)
@@
 			(project "SCCS-RPI"
 				(path "/ce21946f-7655-4864-b48a-50deff8538eb/289c7879-c293-41e1-9b12-36ce1916fe2d"
-					(reference "C46")
+					(reference "C54")
 					(unit 1)
 				)
 				(path "/ce21946f-7655-4864-b48a-50deff8538eb/a0eedc41-812c-454a-9c61-ce155b766160"
-					(reference "C48")
+					(reference "C56")
 					(unit 1)
 				)
 				(path "/ce21946f-7655-4864-b48a-50deff8538eb/a3c5f999-1a2d-4d52-a7d9-976e13506cfb"
-					(reference "C50")
+					(reference "C58")
 					(unit 1)
 				)
 				(path "/ce21946f-7655-4864-b48a-50deff8538eb/f9fe6a99-0547-4304-8cea-93a9433511c0"
-					(reference "C64")
+					(reference "C60")
 					(unit 1)
 				)
@@
 		(dnp no)
 		(fields_autoplaced yes)
-		(property "Reference" "#PWR048"
+		(property "Reference" "#PWR067"
 			(at 96.52 74.93 0)
 			(hide yes)
@@
 			(project "SCCS-RPI"
 				(path "/ce21946f-7655-4864-b48a-50deff8538eb/289c7879-c293-41e1-9b12-36ce1916fe2d"
-					(reference "#PWR048")
+					(reference "#PWR067")
 					(unit 1)
 				)
 				(path "/ce21946f-7655-4864-b48a-50deff8538eb/a0eedc41-812c-454a-9c61-ce155b766160"
-					(reference "#PWR065")
+					(reference "#PWR068")
 					(unit 1)
 				)
 				(path "/ce21946f-7655-4864-b48a-50deff8538eb/a3c5f999-1a2d-4d52-a7d9-976e13506cfb"
-					(reference "#PWR074")
+					(reference "#PWR069")
 					(unit 1)
 				)
 				(path "/ce21946f-7655-4864-b48a-50deff8538eb/f9fe6a99-0547-4304-8cea-93a9433511c0"
-					(reference "#PWR0113")
+					(reference "#PWR070")
 					(unit 1)
 				)
@@
 				)
 				(path "/ce21946f-7655-4864-b48a-50deff8538eb/a0eedc41-812c-454a-9c61-ce155b766160"
-					(reference "D24")
+					(reference "D16")
 					(unit 1)
 				)
 				(path "/ce21946f-7655-4864-b48a-50deff8538eb/a3c5f999-1a2d-4d52-a7d9-976e13506cfb"
-					(reference "D29")
+					(reference "D17")
 					(unit 1)
 				)
 				(path "/ce21946f-7655-4864-b48a-50deff8538eb/f9fe6a99-0547-4304-8cea-93a9433511c0"
-					(reference "D44")
+					(reference "D18")
 					(unit 1)
 				)
@@
 		(in_pos_files yes)
 		(dnp no)
-		(property "Reference" "C47"
+		(property "Reference" "C55"
 			(at 102.616 65.024 0)
 			(show_name no)
@@
 			(project "SCCS-RPI"
 				(path "/ce21946f-7655-4864-b48a-50deff8538eb/289c7879-c293-41e1-9b12-36ce1916fe2d"
-					(reference "C47")
+					(reference "C55")
 					(unit 1)
 				)
 				(path "/ce21946f-7655-4864-b48a-50deff8538eb/a0eedc41-812c-454a-9c61-ce155b766160"
-					(reference "C49")
+					(reference "C57")
 					(unit 1)
 				)
 				(path "/ce21946f-7655-4864-b48a-50deff8538eb/a3c5f999-1a2d-4d52-a7d9-976e13506cfb"
-					(reference "C51")
+					(reference "C59")
 					(unit 1)
 				)
 				(path "/ce21946f-7655-4864-b48a-50deff8538eb/f9fe6a99-0547-4304-8cea-93a9433511c0"
-					(reference "C65")
-					(unit 1)
-				)
+					(reference "C61")
+					(unit 1)
+				)
