File: kicad/reed_input.kicad_sch (KiCad schematic)
At the start: 6 parts

Commit message: Updated Kicad schematics
Parts:
- R21: renamed from R24; value 4.7K -> 220R; LCSC Part # C17673 -> C17557
- renumbered R23 to R20
Changed lines of the file:
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@@
 		(in_pos_files yes)
 		(dnp no)
-		(property "Reference" "R23"
+		(property "Reference" "R20"
 			(at 112.522 63.5 0)
 			(show_name no)
@@
 			(project "SCCS-RPI"
 				(path "/ce21946f-7655-4864-b48a-50deff8538eb/3ce61252-32ee-46c5-9d9c-cf7cd20b8d46"
-					(reference "R29")
+					(reference "R26")
 					(unit 1)
 				)
 				(path "/ce21946f-7655-4864-b48a-50deff8538eb/481789b0-b03f-4fb6-8cab-4075070a7d1e"
-					(reference "R35")
+					(reference "R32")
 					(unit 1)
 				)
 				(path "/ce21946f-7655-4864-b48a-50deff8538eb/572e5cbc-5c13-4858-8c39-64d2a555b72a"
-					(reference "R23")
+					(reference "R20")
 					(unit 1)
 				)
 				(path "/ce21946f-7655-4864-b48a-50deff8538eb/95bed2d0-df43-4056-b799-ae5d23da14c6"
-					(reference "R31")
+					(reference "R28")
 					(unit 1)
 				)
 				(path "/ce21946f-7655-4864-b48a-50deff8538eb/a5503c16-2320-4b38-b3ea-b1cc40d6c763"
-					(reference "R27")
+					(reference "R24")
 					(unit 1)
 				)
 				(path "/ce21946f-7655-4864-b48a-50deff8538eb/eed03f6e-bc4f-485d-9f39-887ce0e6700d"
-					(reference "R33")
+					(reference "R30")
 					(unit 1)
 				)
 				(path "/ce21946f-7655-4864-b48a-50deff8538eb/f0dd22ba-7b40-4c06-b812-0685d925c1df"
-					(reference "R37")
+					(reference "R34")
 					(unit 1)
 				)
 				(path "/ce21946f-7655-4864-b48a-50deff8538eb/f7d9daaf-814c-4f9c-a1f6-c4a86ccfc345"
-					(reference "R25")
+					(reference "R22")
 					(unit 1)
 				)
@@
 		(dnp no)
 		(fields_autoplaced yes)
-		(property "Reference" "#PWR032"
+		(property "Reference" "#PWR033"
 			(at 111.76 57.15 0)
 			(hide yes)
@@
 			(project "SCCS-RPI"
 				(path "/ce21946f-7655-4864-b48a-50deff8538eb/3ce61252-32ee-46c5-9d9c-cf7cd20b8d46"
-					(reference "#PWR038")
+					(reference "#PWR039")
 					(unit 1)
 				)
 				(path "/ce21946f-7655-4864-b48a-50deff8538eb/481789b0-b03f-4fb6-8cab-4075070a7d1e"
-					(reference "#PWR044")
+					(reference "#PWR045")
 					(unit 1)
 				)
 				(path "/ce21946f-7655-4864-b48a-50deff8538eb/572e5cbc-5c13-4858-8c39-64d2a555b72a"
-					(reference "#PWR032")
+					(reference "#PWR033")
 					(unit 1)
 				)
 				(path "/ce21946f-7655-4864-b48a-50deff8538eb/95bed2d0-df43-4056-b799-ae5d23da14c6"
-					(reference "#PWR040")
+					(reference "#PWR041")
 					(unit 1)
 				)
 				(path "/ce21946f-7655-4864-b48a-50deff8538eb/a5503c16-2320-4b38-b3ea-b1cc40d6c763"
-					(reference "#PWR036")
+					(reference "#PWR037")
 					(unit 1)
 				)
 				(path "/ce21946f-7655-4864-b48a-50deff8538eb/eed03f6e-bc4f-485d-9f39-887ce0e6700d"
-					(reference "#PWR042")
+					(reference "#PWR043")
 					(unit 1)
 				)
 				(path "/ce21946f-7655-4864-b48a-50deff8538eb/f0dd22ba-7b40-4c06-b812-0685d925c1df"
-					(reference "#PWR046")
+					(reference "#PWR047")
 					(unit 1)
 				)
 				(path "/ce21946f-7655-4864-b48a-50deff8538eb/f7d9daaf-814c-4f9c-a1f6-c4a86ccfc345"
-					(reference "#PWR034")
+					(reference "#PWR035")
 					(unit 1)
 				)
@@
 		(dnp no)
 		(fields_autoplaced yes)
-		(property "Reference" "#PWR033"
+		(property "Reference" "#PWR034"
 			(at 127 85.09 0)
 			(hide yes)
@@
 			(project "SCCS-RPI"
 				(path "/ce21946f-7655-4864-b48a-50deff8538eb/3ce61252-32ee-46c5-9d9c-cf7cd20b8d46"
-					(reference "#PWR039")
+					(reference "#PWR040")
 					(unit 1)
 				)
 				(path "/ce21946f-7655-4864-b48a-50deff8538eb/481789b0-b03f-4fb6-8cab-4075070a7d1e"
-					(reference "#PWR045")
+					(reference "#PWR046")
 					(unit 1)
 				)
 				(path "/ce21946f-7655-4864-b48a-50deff8538eb/572e5cbc-5c13-4858-8c39-64d2a555b72a"
-					(reference "#PWR033")
+					(reference "#PWR034")
 					(unit 1)
 				)
 				(path "/ce21946f-7655-4864-b48a-50deff8538eb/95bed2d0-df43-4056-b799-ae5d23da14c6"
-					(reference "#PWR041")
+					(reference "#PWR042")
 					(unit 1)
 				)
 				(path "/ce21946f-7655-4864-b48a-50deff8538eb/a5503c16-2320-4b38-b3ea-b1cc40d6c763"
-					(reference "#PWR037")
+					(reference "#PWR038")
 					(unit 1)
 				)
 				(path "/ce21946f-7655-4864-b48a-50deff8538eb/eed03f6e-bc4f-485d-9f39-887ce0e6700d"
-					(reference "#PWR043")
+					(reference "#PWR044")
 					(unit 1)
 				)
 				(path "/ce21946f-7655-4864-b48a-50deff8538eb/f0dd22ba-7b40-4c06-b812-0685d925c1df"
-					(reference "#PWR047")
+					(reference "#PWR048")
 					(unit 1)
 				)
 				(path "/ce21946f-7655-4864-b48a-50deff8538eb/f7d9daaf-814c-4f9c-a1f6-c4a86ccfc345"
-					(reference "#PWR035")
+					(reference "#PWR036")
 					(unit 1)
 				)
@@
 		(in_pos_files yes)
 		(dnp no)
-		(property "Reference" "R24"
+		(property "Reference" "R21"
 			(at 102.616 67.31 90)
 			(show_name no)
@@
 			)
 		)
-		(property "Value" "4.7K"
+		(property "Value" "220R"
 			(at 105.41 66.04 90)
 			(show_name no)
@@
 			)
 		)
-		(property "LCSC Part #" "C17673"
+		(property "LCSC Part #" "C17557"
 			(at 105.41 66.04 90)
 			(hide yes)
@@
 			(project "SCCS-RPI"
 				(path "/ce21946f-7655-4864-b48a-50deff8538eb/3ce61252-32ee-46c5-9d9c-cf7cd20b8d46"
-					(reference "R30")
+					(reference "R27")
 					(unit 1)
 				)
 				(path "/ce21946f-7655-4864-b48a-50deff8538eb/481789b0-b03f-4fb6-8cab-4075070a7d1e"
-					(reference "R36")
+					(reference "R33")
 					(unit 1)
 				)
 				(path "/ce21946f-7655-4864-b48a-50deff8538eb/572e5cbc-5c13-4858-8c39-64d2a555b72a"
-					(reference "R24")
+					(reference "R21")
 					(unit 1)
 				)
 				(path "/ce21946f-7655-4864-b48a-50deff8538eb/95bed2d0-df43-4056-b799-ae5d23da14c6"
-					(reference "R32")
+					(reference "R29")
 					(unit 1)
 				)
 				(path "/ce21946f-7655-4864-b48a-50deff8538eb/a5503c16-2320-4b38-b3ea-b1cc40d6c763"
-					(reference "R28")
+					(reference "R25")
 					(unit 1)
 				)
 				(path "/ce21946f-7655-4864-b48a-50deff8538eb/eed03f6e-bc4f-485d-9f39-887ce0e6700d"
-					(reference "R34")
+					(reference "R31")
 					(unit 1)
 				)
 				(path "/ce21946f-7655-4864-b48a-50deff8538eb/f0dd22ba-7b40-4c06-b812-0685d925c1df"
-					(reference "R38")
+					(reference "R35")
 					(unit 1)
 				)
 				(path "/ce21946f-7655-4864-b48a-50deff8538eb/f7d9daaf-814c-4f9c-a1f6-c4a86ccfc345"
-					(reference "R26")
-					(unit 1)
-				)
+					(reference "R23")
+					(unit 1)
+				)
