File: kicad/relay_channel.kicad_sch (KiCad schematic)
At the start: 12 parts, among them K1 Relay_SPDT, Q13 2N7000, U2 PC817

Commit message: Updated Kicad schematics
Parts:
- renumbered C60 to C62, D32 to D37, D33 to D38, Q13 to Q17, R79 to R90, R80 to R91, R81 to R92, R82 to R93
Changed lines of the file:
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@@
 		(dnp no)
 		(fields_autoplaced yes)
-		(property "Reference" "C60"
+		(property "Reference" "C62"
 			(at 102.8763 39.37 90)
 			(show_name no)
@@
 			(project "SCCS-RPI"
 				(path "/ce21946f-7655-4864-b48a-50deff8538eb/67cc456c-a1bb-42f9-9e79-f18883d18275"
+					(reference "C65")
+					(unit 1)
+				)
+				(path "/ce21946f-7655-4864-b48a-50deff8538eb/6d499a9e-12be-48c7-97b5-aaa8433b7610"
+					(reference "C64")
+					(unit 1)
+				)
+				(path "/ce21946f-7655-4864-b48a-50deff8538eb/b2c53e19-e42b-4380-a3f5-c04d8b1a12f2"
+					(reference "C62")
+					(unit 1)
+				)
+				(path "/ce21946f-7655-4864-b48a-50deff8538eb/f5b14127-5321-4517-88f3-03b8eaf90121"
 					(reference "C63")
-					(unit 1)
-				)
-				(path "/ce21946f-7655-4864-b48a-50deff8538eb/6d499a9e-12be-48c7-97b5-aaa8433b7610"
-					(reference "C62")
-					(unit 1)
-				)
-				(path "/ce21946f-7655-4864-b48a-50deff8538eb/b2c53e19-e42b-4380-a3f5-c04d8b1a12f2"
-					(reference "C60")
-					(unit 1)
-				)
-				(path "/ce21946f-7655-4864-b48a-50deff8538eb/f5b14127-5321-4517-88f3-03b8eaf90121"
-					(reference "C61")
 					(unit 1)
 				)
@@
 		(in_pos_files yes)
 		(dnp no)
-		(property "Reference" "R82"
+		(property "Reference" "R93"
 			(at 85.09 63.246 90)
 			(show_name no)
@@
 			(project "SCCS-RPI"
 				(path "/ce21946f-7655-4864-b48a-50deff8538eb/67cc456c-a1bb-42f9-9e79-f18883d18275"
-					(reference "R94")
+					(reference "R105")
 					(unit 1)
 				)
 				(path "/ce21946f-7655-4864-b48a-50deff8538eb/6d499a9e-12be-48c7-97b5-aaa8433b7610"
-					(reference "R90")
+					(reference "R101")
 					(unit 1)
 				)
 				(path "/ce21946f-7655-4864-b48a-50deff8538eb/b2c53e19-e42b-4380-a3f5-c04d8b1a12f2"
-					(reference "R82")
+					(reference "R93")
 					(unit 1)
 				)
 				(path "/ce21946f-7655-4864-b48a-50deff8538eb/f5b14127-5321-4517-88f3-03b8eaf90121"
-					(reference "R86")
+					(reference "R97")
 					(unit 1)
 				)
@@
 		(in_pos_files yes)
 		(dnp no)
-		(property "Reference" "#PWR094"
+		(property "Reference" "#PWR0106"
 			(at 67.31 64.77 0)
 			(hide yes)
@@
 			(project "SCCS-RPI"
 				(path "/ce21946f-7655-4864-b48a-50deff8538eb/67cc456c-a1bb-42f9-9e79-f18883d18275"
-					(reference "#PWR0103")
+					(reference "#PWR0115")
 					(unit 1)
 				)
 				(path "/ce21946f-7655-4864-b48a-50deff8538eb/6d499a9e-12be-48c7-97b5-aaa8433b7610"
-					(reference "#PWR0100")
+					(reference "#PWR0112")
 					(unit 1)
 				)
 				(path "/ce21946f-7655-4864-b48a-50deff8538eb/b2c53e19-e42b-4380-a3f5-c04d8b1a12f2"
-					(reference "#PWR094")
+					(reference "#PWR0106")
 					(unit 1)
 				)
 				(path "/ce21946f-7655-4864-b48a-50deff8538eb/f5b14127-5321-4517-88f3-03b8eaf90121"
-					(reference "#PWR097")
+					(reference "#PWR0109")
 					(unit 1)
 				)
@@
 		(in_pos_files yes)
 		(dnp no)
-		(property "Reference" "R81"
+		(property "Reference" "R92"
 			(at 99.06 56.134 90)
 			(show_name no)
@@
 			(project "SCCS-RPI"
 				(path "/ce21946f-7655-4864-b48a-50deff8538eb/67cc456c-a1bb-42f9-9e79-f18883d18275"
-					(reference "R93")
+					(reference "R104")
 					(unit 1)
 				)
 				(path "/ce21946f-7655-4864-b48a-50deff8538eb/6d499a9e-12be-48c7-97b5-aaa8433b7610"
-					(reference "R89")
+					(reference "R100")
 					(unit 1)
 				)
 				(path "/ce21946f-7655-4864-b48a-50deff8538eb/b2c53e19-e42b-4380-a3f5-c04d8b1a12f2"
-					(reference "R81")
+					(reference "R92")
 					(unit 1)
 				)
 				(path "/ce21946f-7655-4864-b48a-50deff8538eb/f5b14127-5321-4517-88f3-03b8eaf90121"
-					(reference "R85")
+					(reference "R96")
 					(unit 1)
 				)
@@
 		(dnp no)
 		(fields_autoplaced yes)
-		(property "Reference" "Q13"
+		(property "Reference" "Q17"
 			(at 102.87 72.39 90)
 			(show_name no)
@@
 			(project "SCCS-RPI"
 				(path "/ce21946f-7655-4864-b48a-50deff8538eb/67cc456c-a1bb-42f9-9e79-f18883d18275"
-					(reference "Q16")
+					(reference "Q20")
 					(unit 1)
 				)
 				(path "/ce21946f-7655-4864-b48a-50deff8538eb/6d499a9e-12be-48c7-97b5-aaa8433b7610"
-					(reference "Q15")
+					(reference "Q19")
 					(unit 1)
 				)
 				(path "/ce21946f-7655-4864-b48a-50deff8538eb/b2c53e19-e42b-4380-a3f5-c04d8b1a12f2"
-					(reference "Q13")
+					(reference "Q17")
 					(unit 1)
 				)
 				(path "/ce21946f-7655-4864-b48a-50deff8538eb/f5b14127-5321-4517-88f3-03b8eaf90121"
-					(reference "Q14")
+					(reference "Q18")
 					(unit 1)
 				)
@@
 		(in_pos_files yes)
 		(dnp no)
-		(property "Reference" "#PWR093"
+		(property "Reference" "#PWR0105"
 			(at 133.35 46.99 0)
 			(hide yes)
@@
 			(project "SCCS-RPI"
 				(path "/ce21946f-7655-4864-b48a-50deff8538eb/67cc456c-a1bb-42f9-9e79-f18883d18275"
-					(reference "#PWR0102")
+					(reference "#PWR0114")
 					(unit 1)
 				)
 				(path "/ce21946f-7655-4864-b48a-50deff8538eb/6d499a9e-12be-48c7-97b5-aaa8433b7610"
-					(reference "#PWR099")
+					(reference "#PWR0111")
 					(unit 1)
 				)
 				(path "/ce21946f-7655-4864-b48a-50deff8538eb/b2c53e19-e42b-4380-a3f5-c04d8b1a12f2"
-					(reference "#PWR093")
+					(reference "#PWR0105")
 					(unit 1)
 				)
 				(path "/ce21946f-7655-4864-b48a-50deff8538eb/f5b14127-5321-4517-88f3-03b8eaf90121"
-					(reference "#PWR096")
+					(reference "#PWR0108")
 					(unit 1)
 				)
@@
 		(in_pos_files yes)
 		(dnp no)
-		(property "Reference" "D32"
+		(property "Reference" "D37"
 			(at 129.286 51.562 0)
 			(show_name no)
@@
 			(project "SCCS-RPI"
 				(path "/ce21946f-7655-4864-b48a-50deff8538eb/67cc456c-a1bb-42f9-9e79-f18883d18275"
-					(reference "D38")
+					(reference "D43")
 					(unit 1)
 				)
 				(path "/ce21946f-7655-4864-b48a-50deff8538eb/6d499a9e-12be-48c7-97b5-aaa8433b7610"
-					(reference "D36")
+					(reference "D41")
 					(unit 1)
 				)
 				(path "/ce21946f-7655-4864-b48a-50deff8538eb/b2c53e19-e42b-4380-a3f5-c04d8b1a12f2"
-					(reference "D32")
+					(reference "D37")
 					(unit 1)
 				)
 				(path "/ce21946f-7655-4864-b48a-50deff8538eb/f5b14127-5321-4517-88f3-03b8eaf90121"
-					(reference "D34")
+					(reference "D39")
 					(unit 1)
 				)
@@
 		(in_pos_files yes)
 		(dnp no)
-		(property "Reference" "R79"
+		(property "Reference" "R90"
 			(at 63.5 48.006 90)
 			(show_name no)
@@
 			(project "SCCS-RPI"
 				(path "/ce21946f-7655-4864-b48a-50deff8538eb/67cc456c-a1bb-42f9-9e79-f18883d18275"
-					(reference "R91")
+					(reference "R102")
 					(unit 1)
 				)
 				(path "/ce21946f-7655-4864-b48a-50deff8538eb/6d499a9e-12be-48c7-97b5-aaa8433b7610"
-					(reference "R87")
+					(reference "R98")
 					(unit 1)
 				)
 				(path "/ce21946f-7655-4864-b48a-50deff8538eb/b2c53e19-e42b-4380-a3f5-c04d8b1a12f2"
-					(reference "R79")
+					(reference "R90")
 					(unit 1)
 				)
 				(path "/ce21946f-7655-4864-b48a-50deff8538eb/f5b14127-5321-4517-88f3-03b8eaf90121"
-					(reference "R83")
+					(reference "R94")
 					(unit 1)
 				)
@@
 		(in_pos_files yes)
 		(dnp no)
-		(property "Reference" "R80"
+		(property "Reference" "R91"
 			(at 121.92 52.578 90)
 			(show_name no)
@@
 			(project "SCCS-RPI"
 				(path "/ce21946f-7655-4864-b48a-50deff8538eb/67cc456c-a1bb-42f9-9e79-f18883d18275"
-					(reference "R92")
+					(reference "R103")
 					(unit 1)
 				)
 				(path "/ce21946f-7655-4864-b48a-50deff8538eb/6d499a9e-12be-48c7-97b5-aaa8433b7610"
-					(reference "R88")
+					(reference "R99")
 					(unit 1)
 				)
 				(path "/ce21946f-7655-4864-b48a-50deff8538eb/b2c53e19-e42b-4380-a3f5-c04d8b1a12f2"
-					(reference "R80")
+					(reference "R91")
 					(unit 1)
 				)
 				(path "/ce21946f-7655-4864-b48a-50deff8538eb/f5b14127-5321-4517-88f3-03b8eaf90121"
-					(reference "R84")
+					(reference "R95")
 					(unit 1)
 				)
@@
 		(in_pos_files yes)
 		(dnp no)
-		(property "Reference" "#PWR095"
+		(property "Reference" "#PWR0107"
 			(at 91.44 81.28 0)
 			(hide yes)
@@
 			(project "SCCS-RPI"
 				(path "/ce21946f-7655-4864-b48a-50deff8538eb/67cc456c-a1bb-42f9-9e79-f18883d18275"
-					(reference "#PWR0104")
+					(reference "#PWR0116")
 					(unit 1)
 				)
 				(path "/ce21946f-7655-4864-b48a-50deff8538eb/6d499a9e-12be-48c7-97b5-aaa8433b7610"
-					(reference "#PWR0101")
+					(reference "#PWR0113")
 					(unit 1)
 				)
 				(path "/ce21946f-7655-4864-b48a-50deff8538eb/b2c53e19-e42b-4380-a3f5-c04d8b1a12f2"
-					(reference "#PWR095")
+					(reference "#PWR0107")
 					(unit 1)
 				)
 				(path "/ce21946f-7655-4864-b48a-50deff8538eb/f5b14127-5321-4517-88f3-03b8eaf90121"
-					(reference "#PWR098")
+					(reference "#PWR0110")
 					(unit 1)
 				)
@@
 		(in_pos_files yes)
 		(dnp no)
-		(property "Reference" "D33"
+		(property "Reference" "D38"
 			(at 121.666 57.658 0)
 			(show_name no)
@@
 			(project "SCCS-RPI"
 				(path "/ce21946f-7655-4864-b48a-50deff8538eb/67cc456c-a1bb-42f9-9e79-f18883d18275"
-					(reference "D39")
+					(reference "D44")
 					(unit 1)
 				)
 				(path "/ce21946f-7655-4864-b48a-50deff8538eb/6d499a9e-12be-48c7-97b5-aaa8433b7610"
-					(reference "D37")
+					(reference "D42")
 					(unit 1)
 				)
 				(path "/ce21946f-7655-4864-b48a-50deff8538eb/b2c53e19-e42b-4380-a3f5-c04d8b1a12f2"
-					(reference "D33")
+					(reference "D38")
 					(unit 1)
 				)
 				(path "/ce21946f-7655-4864-b48a-50deff8538eb/f5b14127-5321-4517-88f3-03b8eaf90121"
-					(reference "D35")
-					(unit 1)
-				)
+					(reference "D40")
+					(unit 1)
+				)
