File: kicad/ws2815.kicad_sch (KiCad schematic)
At the start: 2 parts

Commit message: Updated Kicad schematics
Parts:
- renumbered D30 to D35, R75 to R88
Changed lines of the file:
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@@
 		(dnp no)
 		(fields_autoplaced yes)
-		(property "Reference" "#PWR075"
+		(property "Reference" "#PWR0103"
 			(at 160.02 93.98 0)
 			(hide yes)
@@
 			(project "SCCS-RPI"
 				(path "/ce21946f-7655-4864-b48a-50deff8538eb/ca3e75a4-69fa-4118-99c0-ffa695db17b0"
-					(reference "#PWR075")
+					(reference "#PWR0103")
 					(unit 1)
 				)
 				(path "/ce21946f-7655-4864-b48a-50deff8538eb/ecbbfcd6-f58c-4962-8970-f2896585c8c2"
-					(reference "#PWR076")
+					(reference "#PWR0104")
 					(unit 1)
 				)
@@
 		(in_pos_files yes)
 		(dnp no)
-		(property "Reference" "R75"
+		(property "Reference" "R88"
 			(at 149.098 99.314 90)
 			(show_name no)
@@
 			(project "SCCS-RPI"
 				(path "/ce21946f-7655-4864-b48a-50deff8538eb/ca3e75a4-69fa-4118-99c0-ffa695db17b0"
-					(reference "R75")
+					(reference "R88")
 					(unit 1)
 				)
 				(path "/ce21946f-7655-4864-b48a-50deff8538eb/ecbbfcd6-f58c-4962-8970-f2896585c8c2"
-					(reference "R76")
+					(reference "R89")
 					(unit 1)
 				)
@@
 		(dnp no)
 		(fields_autoplaced yes)
-		(property "Reference" "D30"
+		(property "Reference" "D35"
 			(at 157.48 95.2499 90)
 			(show_name no)
@@
 			(project "SCCS-RPI"
 				(path "/ce21946f-7655-4864-b48a-50deff8538eb/ca3e75a4-69fa-4118-99c0-ffa695db17b0"
-					(reference "D30")
+					(reference "D35")
 					(unit 1)
 				)
 				(path "/ce21946f-7655-4864-b48a-50deff8538eb/ecbbfcd6-f58c-4962-8970-f2896585c8c2"
-					(reference "D31")
-					(unit 1)
-				)
+					(reference "D36")
+					(unit 1)
+				)
